Commit message: made a teensy port

File: parol6_hardware/urdf/parol6.ros2_control.xacro (robot description, xacro)
@@ -9,5 +9,5 @@
 -->
 <robot xmlns:xacro="http://www.ros.org/wiki/xacro">
-  <xacro:macro name="parol6_ros2_control" params="name use_sim_time:=false serial_port:=/dev/ttyUSB0 baud_rate:=115200">
+  <xacro:macro name="parol6_ros2_control" params="name use_sim_time:=false serial_port:=/dev/ttyACM0 baud_rate:=115200">
     <!-- ======================================================================
          ros2_control Hardware Interface Configuration

File: parol6_hardware/urdf/parol6.urdf.xacro (robot description, xacro)
@@ -21,5 +21,5 @@
   <!-- Arguments -->
   <xacro:arg name="use_ros2_control" default="true"/>
-  <xacro:arg name="serial_port" default="/dev/ttyUSB0"/>
+  <xacro:arg name="serial_port" default="/dev/ttyACM0"/>
   <xacro:arg name="baud_rate" default="115200"/>
   <!-- ========================================================================

Commit message: feat: Implement configuration validation in the configurator, enhance firmware homing and safety supervisor logic, and add status telemetry.

File: parol6_hardware/urdf/parol6.ros2_control.xacro (robot description, xacro)
@@ -13,5 +13,5 @@
 -->
 <robot xmlns:xacro="http://www.ros.org/wiki/xacro">
-  <xacro:macro name="parol6_ros2_control" params="name use_sim_time:=false serial_port:=/dev/ttyACM0 baud_rate:=115200">
+  <xacro:macro name="parol6_ros2_control" params="name use_sim_time:=false serial_port:=/dev/ttyACM0 baud_rate:=115200 allow_spoofing:=false">
     <!-- ======================================================================
          ros2_control Hardware Interface Configuration
@@ -24,4 +24,5 @@
         <param name="serial_port">${serial_port}</param>
         <param name="baud_rate">${baud_rate}</param>
+        <param name="allow_spoofing">${allow_spoofing}</param>
         <param name="timeout_ms">5</param>        <!-- Must be << loop period (40ms @ 25Hz) -->
         <!-- Logging -->
