Commit message: feat: Refactor parol6_arm_controller parameters in YAML and replace the URDF with a simplified 6-DOF model for Software-in-the-Loop validation.

File: parol6_hardware/urdf/parol6.urdf.xacro (robot description, xacro)
@@ -1,31 +1,137 @@
 <?xml version="1.0"?>
 <!--
-  Main URDF/xacro for PAROL6 with ros2_control
-  Day 1: SIL (Software-in-the-Loop) Validation
-  This file combines:
-  1. Original PAROL6 URDF (robot geometry, visuals, collisions)
-  2. ros2_control hardware interface configuration
+  Day 1 SIL URDF for PAROL6
+  This is a SIMPLIFIED robot model for Software-in-the-Loop validation.
+  Purpose:
+  - Validate ros2_control plumbing without hardware
+  - Test controller loading and activation
+  - Verify /joint_states topic publishing
+  What's included:
+  - Basic kinematic chain (6 revolute joints)
+  - ros2_control hardware interface (PAROL6System only)
+  - Minimal links for TF tree
+  What's NOT included:
+  - Gazebo/Ignition tags (causes IgnitionSystem conflict)
+  - Detailed geometry/meshes
+  - Full PAROL6 URDF (will integrate in Day 2+)
   Usage:
-    xacro parol6.urdf.xacro > parol6_with_ros2_control.urdf
-  Or in launch file:
-    robot_description_content = Command([xacro, " ", xacro_file, " ", "use_ros2_control:=true"])
+    This URDF is automatically loaded by real_robot.launch.py
 -->
 <robot xmlns:xacro="http://www.ros.org/wiki/xacro" name="parol6">
-  <!-- Parameters -->
+  <!-- Arguments -->
   <xacro:arg name="use_ros2_control" default="true"/>
   <xacro:arg name="serial_port" default="/dev/ttyUSB0"/>
   <xacro:arg name="baud_rate" default="115200"/>
   <!-- ========================================================================
-       Include Original PAROL6 URDF
+       BASE ROBOT STRUCTURE (Simplified for Day 1)
        ======================================================================== -->
-  <!-- Xacro can include plain URDF files directly - no conversion needed! -->
-  <xacro:include filename="$(find parol6)/urdf/PAROL6.urdf"/>
+  <!-- Base link -->
+  <link name="base_link">
+    <visual>
+      <geometry>
+        <box size="0.1 0.1 0.05"/>
+      </geometry>
+      <material name="base_material">
+        <color rgba="0.5 0.5 0.5 1.0"/>
+      </material>
+    </visual>
+  </link>
+  <!-- Joint 1 (Base rotation) -->
+  <joint name="joint_L1" type="revolute">
+    <parent link="base_link"/>
+    <child link="link1"/>
+    <origin xyz="0 0 0.05" rpy="0 0 0"/>
+    <axis xyz="0 0 1"/>
+    <limit lower="-3.14" upper="3.14" effort="100" velocity="1.0"/>
+  </joint>
+  <link name="link1">
+    <visual>
+      <geometry>
+        <cylinder radius="0.03" length="0.1"/>
+      </geometry>
+    </visual>
+  </link>
+  <!-- Joint 2 -->
+  <joint name="joint_L2" type="revolute">
+    <parent link="link1"/>
+    <child link="link2"/>
+    <origin xyz="0 0 0.1" rpy="0 0 0"/>
+    <axis xyz="0 1 0"/>
+    <limit lower="-3.14" upper="3.14" effort="100" velocity="1.0"/>
+  </joint>
+  <link name="link2">
+    <visual>
+      <geometry>
+        <cylinder radius="0.025" length="0.15"/>
+      </geometry>
+    </visual>
+  </link>
+  <!-- Joint 3 -->
+  <joint name="joint_L3" type="revolute">
+    <parent link="link2"/>
+    <child link="link3"/>
+    <origin xyz="0 0 0.15" rpy="0 0 0"/>
+    <axis xyz="0 1 0"/>
+    <limit lower="-3.14" upper="3.14" effort="100" velocity="1.0"/>
+  </joint>
+  <link name="link3">
+    <visual>
+      <geometry>
+        <cylinder radius="0.02" length="0.12"/>
+      </geometry>
+    </visual>
+  </link>
+  <!-- Joint 4 -->
+  <joint name="joint_L4" type="revolute">
+    <parent link="link3"/>
+    <child link="link4"/>
+    <origin xyz="0 0 0.12" rpy="0 0 0"/>
+    <axis xyz="1 0 0"/>
+    <limit lower="-3.14" upper="3.14" effort="50" velocity="1.0"/>
+  </joint>
+  <link name="link4">
+    <visual>
+      <geometry>
+        <cylinder radius="0.015" length="0.08"/>
+      </geometry>
+    </visual>
+  </link>
+  <!-- Joint 5 -->
+  <joint name="joint_L5" type="revolute">
+    <parent link="link4"/>
+    <child link="link5"/>
+    <origin xyz="0 0 0.08" rpy="0 0 0"/>
+    <axis xyz="0 1 0"/>
+    <limit lower="-3.14" upper="3.14" effort="50" velocity="1.0"/>
+  </joint>
+  <link name="link5">
+    <visual>
+      <geometry>
+        <cylinder radius="0.015" length="0.06"/>
+      </geometry>
+    </visual>
+  </link>
+  <!-- Joint 6 (End effector rotation) -->
+  <joint name="joint_L6" type="revolute">
+    <parent link="link5"/>
+    <child link="link6"/>
+    <origin xyz="0 0 0.06" rpy="0 0 0"/>
+    <axis xyz="0 0 1"/>
+    <limit lower="-3.14" upper="3.14" effort="30" velocity="1.0"/>
+  </joint>
+  <link name="link6">
+    <visual>
+      <geometry>
+        <cylinder radius="0.01" length="0.03"/>
+      </geometry>
+    </visual>
+  </link>
   <!-- ========================================================================
-       ros2_control Configuration
+       ros2_control HARDWARE INTERFACE (Real robot only)
        ======================================================================== -->
   <xacro:if value="$(arg use_ros2_control)">
-    <!-- Include ros2_control macro -->
+    <!-- Include ros2_control configuration macro -->
     <xacro:include filename="$(find parol6_hardware)/urdf/parol6.ros2_control.xacro"/>
-    <!-- Instantiate hardware interface -->
+    <!-- Instantiate hardware interface (PAROL6System ONLY - no Gazebo) -->
     <xacro:parol6_ros2_control name="PAROL6Hardware" serial_port="$(arg serial_port)" baud_rate="$(arg baud_rate)"/>
   </xacro:if>

Commit message: feat: Implement telemetry state byte, configurable baud rate, dynamic xacro inversion, and update URDF to full CAD model.

File: parol6_hardware/urdf/parol6.urdf.xacro (robot description, xacro)
@@ -23,108 +23,9 @@
   <xacro:arg name="serial_port" default="/dev/ttyACM0"/>
   <xacro:arg name="baud_rate" default="115200"/>
+  <xacro:arg name="allow_spoofing" default="false"/>
   <!-- ========================================================================
-       BASE ROBOT STRUCTURE (Simplified for Day 1)
+       BASE ROBOT STRUCTURE (Full CAD definitions)
        ======================================================================== -->
-  <!-- Base link -->
-  <link name="base_link">
-    <visual>
-      <geometry>
-        <box size="0.1 0.1 0.05"/>
-      </geometry>
-      <material name="base_material">
-        <color rgba="0.5 0.5 0.5 1.0"/>
-      </material>
-    </visual>
-  </link>
-  <!-- Joint 1 (Base rotation) -->
-  <joint name="joint_L1" type="revolute">
-    <parent link="base_link"/>
-    <child link="link1"/>
-    <origin xyz="0 0 0.05" rpy="0 0 0"/>
-    <axis xyz="0 0 1"/>
-    <limit lower="-3.14" upper="3.14" effort="100" velocity="1.0"/>
-  </joint>
-  <link name="link1">
-    <visual>
-      <geometry>
-        <cylinder radius="0.03" length="0.1"/>
-      </geometry>
-    </visual>
-  </link>
-  <!-- Joint 2 -->
-  <joint name="joint_L2" type="revolute">
-    <parent link="link1"/>
-    <child link="link2"/>
-    <origin xyz="0 0 0.1" rpy="0 0 0"/>
-    <axis xyz="0 1 0"/>
-    <limit lower="-3.14" upper="3.14" effort="100" velocity="1.0"/>
-  </joint>
-  <link name="link2">
-    <visual>
-      <geometry>
-        <cylinder radius="0.025" length="0.15"/>
-      </geometry>
-    </visual>
-  </link>
-  <!-- Joint 3 -->
-  <joint name="joint_L3" type="revolute">
-    <parent link="link2"/>
-    <child link="link3"/>
-    <origin xyz="0 0 0.15" rpy="0 0 0"/>
-    <axis xyz="0 1 0"/>
-    <limit lower="-3.14" upper="3.14" effort="100" velocity="1.0"/>
-  </joint>
-  <link name="link3">
-    <visual>
-      <geometry>
-        <cylinder radius="0.02" length="0.12"/>
-      </geometry>
-    </visual>
-  </link>
-  <!-- Joint 4 -->
-  <joint name="joint_L4" type="revolute">
-    <parent link="link3"/>
-    <child link="link4"/>
-    <origin xyz="0 0 0.12" rpy="0 0 0"/>
-    <axis xyz="1 0 0"/>
-    <limit lower="-3.14" upper="3.14" effort="50" velocity="1.0"/>
-  </joint>
-  <link name="link4">
-    <visual>
-      <geometry>
-        <cylinder radius="0.015" length="0.08"/>
-      </geometry>
-    </visual>
-  </link>
-  <!-- Joint 5 -->
-  <joint name="joint_L5" type="revolute">
-    <parent link="link4"/>
-    <child link="link5"/>
-    <origin xyz="0 0 0.08" rpy="0 0 0"/>
-    <axis xyz="0 1 0"/>
-    <limit lower="-3.14" upper="3.14" effort="50" velocity="1.0"/>
-  </joint>
-  <link name="link5">
-    <visual>
-      <geometry>
-        <cylinder radius="0.015" length="0.06"/>
-      </geometry>
-    </visual>
-  </link>
-  <!-- Joint 6 (End effector rotation) -->
-  <joint name="joint_L6" type="revolute">
-    <parent link="link5"/>
-    <child link="link6"/>
-    <origin xyz="0 0 0.06" rpy="0 0 0"/>
-    <axis xyz="0 0 1"/>
-    <limit lower="-3.14" upper="3.14" effort="30" velocity="1.0"/>
-  </joint>
-  <link name="link6">
-    <visual>
-      <geometry>
-        <cylinder radius="0.01" length="0.03"/>
-      </geometry>
-    </visual>
-  </link>
+  <xacro:include filename="$(find parol6)/urdf/PAROL6.urdf"/>
   <!-- ========================================================================
        ros2_control HARDWARE INTERFACE (Real robot only)
@@ -134,5 +35,5 @@
     <xacro:include filename="$(find parol6_hardware)/urdf/parol6.ros2_control.xacro"/>
     <!-- Instantiate hardware interface (PAROL6System ONLY - no Gazebo) -->
-    <xacro:parol6_ros2_control name="PAROL6Hardware" serial_port="$(arg serial_port)" baud_rate="$(arg baud_rate)"/>
+    <xacro:parol6_ros2_control name="PAROL6Hardware" serial_port="$(arg serial_port)" baud_rate="$(arg baud_rate)" allow_spoofing="$(arg allow_spoofing)"/>
   </xacro:if>
 </robot>

Commit message: Added missing URDF File

File: parol6_hardware/urdf/parol6.urdf.xacro (robot description, xacro)
@@ -28,4 +28,11 @@
        ======================================================================== -->
   <xacro:include filename="$(find parol6)/urdf/PAROL6.urdf"/>
+  <!-- Dummy link representing the Tool Center Point (TCP) / Gripper Tip -->
+  <link name="tcp_link"/>
+  <joint name="tcp_joint" type="fixed">
+    <origin xyz="0 0 0.1" rpy="0 0 0" />
+    <parent link="link6"/>
+    <child link="tcp_link"/>
+  </joint>
   <!-- ========================================================================
        ros2_control HARDWARE INTERFACE (Real robot only)
