Commit message: Adjusted URDF joint limit of J2 at home position to Match Hardware Limit.

File: PAROL6/urdf/PAROL6.urdf (robot description, URDF)
Before this commit: robot parol6, 8 links, 7 joints
Joints:
- joint joint_L2: limit lower=-0.98 upper=1 effort=300 velocity=3 -> lower=-0.802444444 upper=1 effort=300 velocity=3

Commit message: Updated URDF actual Hardware Limits.

File: PAROL6/urdf/PAROL6.urdf (robot description, URDF)
Before this commit: robot parol6, 8 links, 7 joints
Joints:
- joint joint_L3: limit lower=-2 upper=1.3 effort=300 velocity=3 -> lower=-2 upper=1.186823892 effort=300 velocity=3

Commit message: Updated J4 Actual Hardware Limits.

File: PAROL6/urdf/PAROL6.urdf (robot description, URDF)
Before this commit: robot parol6, 8 links, 7 joints
Joints:
- joint joint_L4: limit lower=-2 upper=2 effort=300 velocity=3 -> lower=-2.4945 upper=1.849111111 effort=300 velocity=3

Commit message: Adjusted J1 Limits.

File: PAROL6/urdf/PAROL6.urdf (robot description, URDF)
Before this commit: robot parol6, 8 links, 7 joints
Joints:
- joint joint_L1: limit lower=-1.7 upper=1.7 effort=300 velocity=3 -> lower=-2.041 upper=1.343 effort=300 velocity=3

Commit message: Updated J1 Limits.

File: PAROL6/urdf/PAROL6.urdf (robot description, URDF)
Before this commit: robot parol6, 8 links, 7 joints
Joints:
- joint joint_L1: limit lower=-1.7 upper=1.7 effort=300 velocity=3 -> lower=-2.045 upper=1.343 effort=300 velocity=3

Commit message: Update J1 Limits v1.2

File: PAROL6/urdf/PAROL6.urdf (robot description, URDF)
Before this commit: robot parol6, 8 links, 7 joints
Joints:
- joint joint_L1: limit lower=-2.045 upper=1.343 effort=300 velocity=3 -> lower=-1.7 upper=1.7 effort=300 velocity=3

Commit message: Updated J1 limits v1.2

File: PAROL6/urdf/PAROL6.urdf (robot description, URDF)
Before this commit: robot parol6, 8 links, 7 joints
Joints:
- joint joint_L1: limit lower=-2.041 upper=1.343 effort=300 velocity=3 -> lower=-1.7 upper=1.7 effort=300 velocity=3

Commit message: Added end effector frame for URDF files.

File: PAROL6/urdf/PAROL6.urdf (robot description, URDF)
Before this commit: robot parol6, 8 links, 7 joints
Links:
- added link tcp_link
Joints:
- added joint tcp_joint: type fixed, parent L6, child tcp_link, origin xyz=0 0 0.1 rpy=0 0 0

File: parol6_hardware/urdf/parol6.urdf.xacro (robot description, xacro)
@@ -127,4 +127,11 @@
     </visual>
   </link>
+  <!-- Dummy link representing the Tool Center Point (TCP) / Gripper Tip -->
+  <link name="tcp_link"/>
+  <joint name="tcp_joint" type="fixed">
+    <origin xyz="0 0 0.1" rpy="0 0 0" />
+    <parent link="link6"/>
+    <child link="tcp_link"/>
+  </joint>
   <!-- ========================================================================
        ros2_control HARDWARE INTERFACE (Real robot only)

Commit message: Updated URDF to take account of an end effector frame.

File: PAROL6/urdf/PAROL6.urdf (robot description, URDF)
Before this commit: robot parol6, 8 links, 7 joints
Links:
- added link tcp_link
Joints:
- added joint tcp_joint: type fixed, parent L6, child tcp_link, origin xyz=0 0 0.1 rpy=0 0 0

Commit message: Added TCP Link to TF links

File: PAROL6/urdf/PAROL6.urdf (robot description, URDF)
Before this commit: robot parol6, 9 links, 8 joints
Links:
- link tcp_link: geometry visual sphere radius=0.01
Joints:
- joint tcp_joint: origin xyz=0 0 0.1 rpy=0 0 0 -> xyz=0 0 0.06 rpy=0 0 0

File: PAROL6/urdf/PAROL6_gazebo.urdf (robot description, URDF)
Before this commit: robot parol6, 8 links, 7 joints
Links:
- added link tcp_link; visual sphere radius=0.01
Joints:
- added joint tcp_joint: type fixed, parent L6, child tcp_link, origin xyz=0 0 0.06 rpy=0 0 0
- joint joint_L6: limit effort=300 velocity=3 -> (none)

File: parol6_hardware/urdf/parol6.urdf.xacro (robot description, xacro)
@@ -28,11 +28,4 @@
        ======================================================================== -->
   <xacro:include filename="$(find parol6)/urdf/PAROL6.urdf"/>
-  <!-- Dummy link representing the Tool Center Point (TCP) / Gripper Tip -->
-  <link name="tcp_link"/>
-  <joint name="tcp_joint" type="fixed">
-    <origin xyz="0 0 0.1" rpy="0 0 0" />
-    <parent link="link6"/>
-    <child link="tcp_link"/>
-  </joint>
   <!-- ========================================================================
        ros2_control HARDWARE INTERFACE (Real robot only)

Commit message: Added Link TCP as end effector

File: PAROL6/urdf/PAROL6.urdf (robot description, URDF)
Before this commit: robot parol6, 8 links, 7 joints
Links:
- added link tcp_link; visual sphere radius=0.01
Joints:
- added joint tcp_joint: type fixed, parent L6, child tcp_link, origin xyz=0 0 -0.075 rpy=0 0 0

Commit message: Fixed Hardware launch method issue

File: PAROL6/urdf/PAROL6.urdf (robot description, URDF)
Before this commit: robot parol6, 9 links, 8 joints
Joints:
- joint tcp_joint: origin xyz=0 0 0.06 rpy=0 0 0 -> xyz=0 0 -0.075 rpy=0 0 0

Commit message: Fixed URDF TCP end effector Rotation bug which causes planning to fail.

File: PAROL6/urdf/PAROL6.urdf (robot description, URDF)
Before this commit: robot parol6, 9 links, 8 joints
Joints:
- joint tcp_joint: origin xyz=0 0 -0.075 rpy=0 0 0 -> xyz=0 0 -0.075 rpy=3.14159 0 0

File: PAROL6/urdf/PAROL6_gazebo.urdf (robot description, URDF)
Before this commit: robot parol6, 9 links, 8 joints
Joints:
- joint tcp_joint: origin xyz=0 0 0.06 rpy=0 0 0 -> xyz=0 0 -0.075 rpy=3.14159 0 0

File: PAROL6/urdf/PAROL6_ignition.urdf (robot description, URDF)
Before this commit: robot parol6, 9 links, 8 joints
Joints:
- joint tcp_joint: origin xyz=0 0 -0.075 rpy=0 0 0 -> xyz=0 0 -0.075 rpy=3.14159 0 0

Commit message: merge

File: PAROL6/urdf/PAROL6.urdf (robot description, URDF)
Before this commit: robot parol6, 8 links, 7 joints
Links:
- added link tcp_link; visual sphere radius=0.01
Joints:
- added joint tcp_joint: type fixed, parent L6, child tcp_link, origin xyz=0 0 -0.075 rpy=3.14159 0 0
- joint joint_L2: limit lower=-0.98 upper=1 effort=300 velocity=3 -> lower=-0.802444444 upper=1 effort=300 velocity=3
- joint joint_L3: limit lower=-2 upper=1.3 effort=300 velocity=3 -> lower=-2 upper=1.186823892 effort=300 velocity=3
- joint joint_L4: limit lower=-2 upper=2 effort=300 velocity=3 -> lower=-2.4945 upper=1.849111111 effort=300 velocity=3

File: PAROL6/urdf/PAROL6_gazebo.urdf (robot description, URDF)
Before this commit: robot parol6, 8 links, 7 joints
Links:
- added link tcp_link; visual sphere radius=0.01
Joints:
- added joint tcp_joint: type fixed, parent L6, child tcp_link, origin xyz=0 0 -0.075 rpy=3.14159 0 0
- joint joint_L6: limit effort=300 velocity=3 -> (none)

File: PAROL6/urdf/PAROL6_ignition.urdf (robot description, URDF)
Before this commit: robot parol6, 8 links, 7 joints
Links:
- added link tcp_link; visual sphere radius=0.01
Joints:
- added joint tcp_joint: type fixed, parent L6, child tcp_link, origin xyz=0 0 -0.075 rpy=3.14159 0 0

Commit message: Optimize Cartesian motion: densify trajectory, sync joint limits, and tune TCP offsets

File: PAROL6/urdf/PAROL6.urdf (robot description, URDF)
Before this commit: robot parol6, 9 links, 8 joints
Joints:
- joint joint_L3: limit lower=-2 upper=1.186823892 effort=300 velocity=3 -> lower=-2 upper=1.29 effort=300 velocity=3
- joint joint_L4: limit lower=-2.4945 upper=1.849111111 effort=300 velocity=3 -> lower=-2.5294444 upper=1.849111111 effort=300 velocity=3
- joint joint_L6: limit effort=300 velocity=3 -> lower=-6.28318 upper=6.28318 effort=300 velocity=3; type continuous -> revolute
- joint tcp_joint: origin xyz=0 0 -0.075 rpy=3.14159 0 0 -> xyz=0 0 -0.1995 rpy=3.14159 0 0

File: PAROL6/urdf/PAROL6_gazebo.urdf (robot description, URDF)
Before this commit: robot parol6, 9 links, 8 joints
Joints:
- joint joint_L6: limit (none) -> lower=-6.28318 upper=6.28318 effort=300 velocity=3; type continuous -> revolute

File: PAROL6/urdf/PAROL6_ignition.urdf (robot description, URDF)
Before this commit: robot parol6, 9 links, 8 joints
Joints:
- joint joint_L6: limit effort=300 velocity=3 -> lower=-6.28318 upper=6.28318 effort=300 velocity=3; type continuous -> revolute

Commit message: Enhanced Tracjectory injection following (Moveit_Controller).

File: PAROL6/urdf/PAROL6.urdf (robot description, URDF)
Before this commit: robot parol6, 9 links, 8 joints
Joints:
- joint tcp_joint: origin xyz=0 0 -0.1995 rpy=3.14159 0 0 -> xyz=-0.0 0.0 -0.09 rpy=3.14159 0 0
